Commit message: more renames

File: rens_description/urdf/2wd_properties.urdf.xacro (robot description, xacro)
@@ -7,5 +7,5 @@
   <!-- set empty on the wheel_mesh_file to use geometry instead of mesh -->
   <xacro:property name="base_mesh_file" value="" />
-  <!-- <xacro:property name="base_mesh_file" value="file://$(find linorobot2_description)/meshes/base.dae" /> -->
+  <!-- <xacro:property name="base_mesh_file" value="file://$(find rens_description)/meshes/base.dae" /> -->
   <xacro:property name="wheel_radius" value="0.072" />
   <xacro:property name="wheel_width" value="0.029" />
@@ -19,5 +19,5 @@
   <!-- set empty on the wheel_mesh_file to use geometry instead of mesh -->
   <xacro:property name="wheel_mesh_file" value="" />
-  <!-- <xacro:property name="wheel_mesh_file" value="file://$(find linorobot2_description)/meshes/tire.dae" /> -->
+  <!-- <xacro:property name="wheel_mesh_file" value="file://$(find rens_description)/meshes/tire.dae" /> -->
   <xacro:property name="laser_pose">
     <origin xyz="0 0 0.08" rpy="0 0 ${pi}"/>

File: rens_description/urdf/4wd_properties.urdf.xacro (robot description, xacro)
@@ -7,5 +7,5 @@
   <!-- set empty on the wheel_mesh_file to use geometry instead of mesh -->
   <xacro:property name="base_mesh_file" value="" />
-  <!-- <xacro:property name="base_mesh_file" value="file://$(find linorobot2_description)/meshes/base.dae" /> -->
+  <!-- <xacro:property name="base_mesh_file" value="file://$(find rens_description)/meshes/base.dae" /> -->
   <xacro:property name="wheel_radius" value="0.07162" />
   <xacro:property name="wheel_width" value="0.05" />
@@ -17,5 +17,5 @@
   <!-- set empty on the wheel_mesh_file to use geometry instead of mesh -->
   <xacro:property name="wheel_mesh_file" value="" />
-  <!-- <xacro:property name="wheel_mesh_file" value="file://$(find linorobot2_description)/meshes/tire.dae" /> -->
+  <!-- <xacro:property name="wheel_mesh_file" value="file://$(find rens_description)/meshes/tire.dae" /> -->
   <xacro:property name="laser_pose">
     <origin xyz="-0.0475 0 0.125" rpy="0 0 0"/>

File: rens_description/urdf/mecanum_properties.urdf.xacro (robot description, xacro)
@@ -7,5 +7,5 @@
   <!-- set empty on the wheel_mesh_file to use geometry instead of mesh -->
   <xacro:property name="base_mesh_file" value="" />
-  <!-- <xacro:property name="base_mesh_file" value="file://$(find linorobot2_description)/meshes/base.dae" /> -->
+  <!-- <xacro:property name="base_mesh_file" value="file://$(find rens_description)/meshes/base.dae" /> -->
   <xacro:property name="wheel_radius" value="0.07162" />
   <xacro:property name="wheel_width" value="0.05" />
@@ -17,5 +17,5 @@
   <!-- set empty on the wheel_mesh_file to use geometry instead of mesh -->
   <xacro:property name="wheel_mesh_file" value="" />
-  <!-- <xacro:property name="wheel_mesh_file" value="file://$(find linorobot2_description)/meshes/tire.dae" /> -->
+  <!-- <xacro:property name="wheel_mesh_file" value="file://$(find rens_description)/meshes/tire.dae" /> -->
   <xacro:property name="laser_pose">
     <origin xyz="-0.0475 0 0.125" rpy="0 0 0"/>

File: rens_description/urdf/robots/2wd.urdf.xacro (robot description, xacro)
@@ -1,14 +1,14 @@
 <?xml version="1.0"?>
-<robot name="linorobot2_2wd" xmlns:xacro="http://ros.org/wiki/xacro">
+<robot name="rens_2wd" xmlns:xacro="http://ros.org/wiki/xacro">
   <xacro:arg name="sim" default="false" />
-  <xacro:include filename="$(find linorobot2_description)/urdf/2wd_properties.urdf.xacro" />
-  <xacro:include filename="$(find linorobot2_description)/urdf/mech/base.urdf.xacro" />
-  <xacro:include filename="$(find linorobot2_description)/urdf/mech/wheel.urdf.xacro" />
-  <xacro:include filename="$(find linorobot2_description)/urdf/mech/caster_wheel.urdf.xacro" />
-  <xacro:include filename="$(find linorobot2_description)/urdf/sensors/plugins.urdf.xacro" />
-  <xacro:include filename="$(find linorobot2_description)/urdf/sensors/imu.urdf.xacro" />
-  <xacro:include filename="$(find linorobot2_description)/urdf/sensors/generic_laser.urdf.xacro" />
-  <xacro:include filename="$(find linorobot2_description)/urdf/sensors/depth_sensor.urdf.xacro" />
-  <xacro:include filename="$(find linorobot2_description)/urdf/controllers/diff_drive.urdf.xacro" />
+  <xacro:include filename="$(find rens_description)/urdf/2wd_properties.urdf.xacro" />
+  <xacro:include filename="$(find rens_description)/urdf/mech/base.urdf.xacro" />
+  <xacro:include filename="$(find rens_description)/urdf/mech/wheel.urdf.xacro" />
+  <xacro:include filename="$(find rens_description)/urdf/mech/caster_wheel.urdf.xacro" />
+  <xacro:include filename="$(find rens_description)/urdf/sensors/plugins.urdf.xacro" />
+  <xacro:include filename="$(find rens_description)/urdf/sensors/imu.urdf.xacro" />
+  <xacro:include filename="$(find rens_description)/urdf/sensors/generic_laser.urdf.xacro" />
+  <xacro:include filename="$(find rens_description)/urdf/sensors/depth_sensor.urdf.xacro" />
+  <xacro:include filename="$(find rens_description)/urdf/controllers/diff_drive.urdf.xacro" />
   <xacro:base
     length="${base_length}"

File: rens_description/urdf/robots/4wd.urdf.xacro (robot description, xacro)
@@ -1,12 +1,12 @@
 <?xml version="1.0"?>
-<robot name="linorobot2_4wd" xmlns:xacro="http://ros.org/wiki/xacro">
-  <xacro:include filename="$(find linorobot2_description)/urdf/4wd_properties.urdf.xacro" />
-  <xacro:include filename="$(find linorobot2_description)/urdf/mech/base.urdf.xacro" />
-  <xacro:include filename="$(find linorobot2_description)/urdf/mech/wheel.urdf.xacro" />
-  <xacro:include filename="$(find linorobot2_description)/urdf/sensors/plugins.urdf.xacro" />
-  <xacro:include filename="$(find linorobot2_description)/urdf/sensors/imu.urdf.xacro" />
-  <xacro:include filename="$(find linorobot2_description)/urdf/sensors/generic_laser.urdf.xacro" />
-  <xacro:include filename="$(find linorobot2_description)/urdf/sensors/depth_sensor.urdf.xacro" />
-  <xacro:include filename="$(find linorobot2_description)/urdf/controllers/skid_steer.urdf.xacro" />
+<robot name="rens_4wd" xmlns:xacro="http://ros.org/wiki/xacro">
+  <xacro:include filename="$(find rens_description)/urdf/4wd_properties.urdf.xacro" />
+  <xacro:include filename="$(find rens_description)/urdf/mech/base.urdf.xacro" />
+  <xacro:include filename="$(find rens_description)/urdf/mech/wheel.urdf.xacro" />
+  <xacro:include filename="$(find rens_description)/urdf/sensors/plugins.urdf.xacro" />
+  <xacro:include filename="$(find rens_description)/urdf/sensors/imu.urdf.xacro" />
+  <xacro:include filename="$(find rens_description)/urdf/sensors/generic_laser.urdf.xacro" />
+  <xacro:include filename="$(find rens_description)/urdf/sensors/depth_sensor.urdf.xacro" />
+  <xacro:include filename="$(find rens_description)/urdf/controllers/skid_steer.urdf.xacro" />
   <xacro:base
     length="${base_length}"

File: rens_description/urdf/robots/mecanum.urdf.xacro (robot description, xacro)
@@ -1,12 +1,12 @@
 <?xml version="1.0"?>
-<robot name="linorobot2_mecanum" xmlns:xacro="http://ros.org/wiki/xacro">
-  <xacro:include filename="$(find linorobot2_description)/urdf/mecanum_properties.urdf.xacro" />
-  <xacro:include filename="$(find linorobot2_description)/urdf/mech/base.urdf.xacro" />
-  <xacro:include filename="$(find linorobot2_description)/urdf/mech/mecanum_wheel.urdf.xacro" />
-  <xacro:include filename="$(find linorobot2_description)/urdf/sensors/plugins.urdf.xacro" />
-  <xacro:include filename="$(find linorobot2_description)/urdf/sensors/imu.urdf.xacro" />
-  <xacro:include filename="$(find linorobot2_description)/urdf/sensors/generic_laser.urdf.xacro" />
-  <xacro:include filename="$(find linorobot2_description)/urdf/sensors/depth_sensor.urdf.xacro" />
-  <xacro:include filename="$(find linorobot2_description)/urdf/controllers/omni_drive.urdf.xacro" />
+<robot name="rens_mecanum" xmlns:xacro="http://ros.org/wiki/xacro">
+  <xacro:include filename="$(find rens_description)/urdf/mecanum_properties.urdf.xacro" />
+  <xacro:include filename="$(find rens_description)/urdf/mech/base.urdf.xacro" />
+  <xacro:include filename="$(find rens_description)/urdf/mech/mecanum_wheel.urdf.xacro" />
+  <xacro:include filename="$(find rens_description)/urdf/sensors/plugins.urdf.xacro" />
+  <xacro:include filename="$(find rens_description)/urdf/sensors/imu.urdf.xacro" />
+  <xacro:include filename="$(find rens_description)/urdf/sensors/generic_laser.urdf.xacro" />
+  <xacro:include filename="$(find rens_description)/urdf/sensors/depth_sensor.urdf.xacro" />
+  <xacro:include filename="$(find rens_description)/urdf/controllers/omni_drive.urdf.xacro" />
   <xacro:base
     length="${base_length}"

File: rens_description/urdf/robots/turtlebot.urdf.xacro (robot description, xacro)
@@ -1,4 +1,4 @@
 <?xml version="1.0"?>
-<robot name="linorobot2_2wd" xmlns:xacro="http://ros.org/wiki/xacro">
+<robot name="rens_2wd" xmlns:xacro="http://ros.org/wiki/xacro">
   <xacro:property name="base_length" value="0.34" />
   <xacro:property name="base_width" value="0.34" />
@@ -14,11 +14,11 @@
   <xacro:property name="front_caster_wheel" value="true" />
   <xacro:property name="rear_caster_wheel" value="true" />
-  <xacro:include filename="$(find linorobot2_description)/urdf/mech/base.urdf.xacro" />
-  <xacro:include filename="$(find linorobot2_description)/urdf/mech/wheel.urdf.xacro" />
-  <xacro:include filename="$(find linorobot2_description)/urdf/mech/caster_wheel.urdf.xacro" />
-  <xacro:include filename="$(find linorobot2_description)/urdf/sensors/imu.urdf.xacro" />
-  <xacro:include filename="$(find linorobot2_description)/urdf/sensors/generic_laser.urdf.xacro" />
-  <xacro:include filename="$(find linorobot2_description)/urdf/sensors/depth_sensor.urdf.xacro" />
-  <xacro:include filename="$(find linorobot2_description)/urdf/controllers/diff_drive.urdf.xacro" />
+  <xacro:include filename="$(find rens_description)/urdf/mech/base.urdf.xacro" />
+  <xacro:include filename="$(find rens_description)/urdf/mech/wheel.urdf.xacro" />
+  <xacro:include filename="$(find rens_description)/urdf/mech/caster_wheel.urdf.xacro" />
+  <xacro:include filename="$(find rens_description)/urdf/sensors/imu.urdf.xacro" />
+  <xacro:include filename="$(find rens_description)/urdf/sensors/generic_laser.urdf.xacro" />
+  <xacro:include filename="$(find rens_description)/urdf/sensors/depth_sensor.urdf.xacro" />
+  <xacro:include filename="$(find rens_description)/urdf/controllers/diff_drive.urdf.xacro" />
   <xacro:property name="laser_pose">
     <origin xyz="0.055 0.02 0.41" rpy="0 0 0"/>

File: rens_description/urdf/robots/vattenkar.urdf.xacro (robot description, xacro)
@@ -1,4 +1,4 @@
 <?xml version="1.0"?>
-<robot name="linorobot2_2wd" xmlns:xacro="http://ros.org/wiki/xacro">
+<robot name="rens_2wd" xmlns:xacro="http://ros.org/wiki/xacro">
   <xacro:property name="base_length" value="0.338" />
   <xacro:property name="base_width" value="0.32" />
@@ -7,5 +7,5 @@
   <!-- set empty on the wheel_mesh_file to use geometry instead of mesh -->
   <xacro:property name="base_mesh_file" value="" />
-  <!-- <xacro:property name="base_mesh_file" value="file://$(find linorobot2_description)/meshes/base.dae" /> -->
+  <!-- <xacro:property name="base_mesh_file" value="file://$(find rens_description)/meshes/base.dae" /> -->
   <xacro:property name="wheel_radius" value="0.0675" />
   <xacro:property name="wheel_width" value="0.022" />
@@ -19,12 +19,12 @@
   <!-- set empty on the wheel_mesh_file to use geometry instead of mesh -->
   <xacro:property name="wheel_mesh_file" value="" />
-  <!-- <xacro:property name="wheel_mesh_file" value="file://$(find linorobot2_description)/meshes/tire.dae" /> -->
-  <xacro:include filename="$(find linorobot2_description)/urdf/mech/base.urdf.xacro" />
-  <xacro:include filename="$(find linorobot2_description)/urdf/mech/wheel.urdf.xacro" />
-  <xacro:include filename="$(find linorobot2_description)/urdf/mech/caster_wheel.urdf.xacro" />
-  <xacro:include filename="$(find linorobot2_description)/urdf/sensors/imu.urdf.xacro" />
-  <xacro:include filename="$(find linorobot2_description)/urdf/sensors/generic_laser.urdf.xacro" />
-  <xacro:include filename="$(find linorobot2_description)/urdf/sensors/depth_sensor.urdf.xacro" />
-  <xacro:include filename="$(find linorobot2_description)/urdf/controllers/diff_drive.urdf.xacro" />
+  <!-- <xacro:property name="wheel_mesh_file" value="file://$(find rens_description)/meshes/tire.dae" /> -->
+  <xacro:include filename="$(find rens_description)/urdf/mech/base.urdf.xacro" />
+  <xacro:include filename="$(find rens_description)/urdf/mech/wheel.urdf.xacro" />
+  <xacro:include filename="$(find rens_description)/urdf/mech/caster_wheel.urdf.xacro" />
+  <xacro:include filename="$(find rens_description)/urdf/sensors/imu.urdf.xacro" />
+  <xacro:include filename="$(find rens_description)/urdf/sensors/generic_laser.urdf.xacro" />
+  <xacro:include filename="$(find rens_description)/urdf/sensors/depth_sensor.urdf.xacro" />
+  <xacro:include filename="$(find rens_description)/urdf/controllers/diff_drive.urdf.xacro" />
   <xacro:property name="laser_pose">
     <origin xyz="0.126 0 0.25" rpy="0 0 -0.78539816339"/>

File: rens_description/urdf/sensors/generic_laser.urdf.xacro (robot description, xacro)
@@ -1,5 +1,5 @@
 <?xml version="1.0"?>
 <robot xmlns:xacro="http://ros.org/wiki/xacro">
-  <xacro:include filename="$(find linorobot2_description)/urdf/sensors/laser.urdf.xacro" />
+  <xacro:include filename="$(find rens_description)/urdf/sensors/laser.urdf.xacro" />
   <xacro:macro name="generic_laser" params="*origin">
     <xacro:laser
