Commit message: eerste stappjes naar het omzetten van URDF naar de REnS

File: linorobot2_description/urdf/2wd_properties.urdf.xacro (robot description, xacro)
@@ -1,19 +1,19 @@
 <?xml version="1.0"?>
 <robot xmlns:xacro="http://ros.org/wiki/xacro">
-  <xacro:property name="base_length" value="0.24" />
-  <xacro:property name="base_width" value="0.275" />
-  <xacro:property name="base_height" value="0.003" />
+  <xacro:property name="base_length" value="0.35" />
+  <xacro:property name="base_width" value="0.230" />
+  <xacro:property name="base_height" value="0.080" />
   <xacro:property name="base_mass" value="1" />
   <!-- set empty on the wheel_mesh_file to use geometry instead of mesh -->
   <xacro:property name="base_mesh_file" value="" />
   <!-- <xacro:property name="base_mesh_file" value="file://$(find linorobot2_description)/meshes/base.dae" /> -->
-  <xacro:property name="wheel_radius" value="0.045" />
-  <xacro:property name="wheel_width" value="0.01" />
-  <xacro:property name="wheel_pos_x" value="0.0" />
-  <xacro:property name="wheel_pos_y" value="0.13" />
+  <xacro:property name="wheel_radius" value="0.072" />
+  <xacro:property name="wheel_width" value="0.029" />
+  <xacro:property name="wheel_pos_x" value="0.09" />
+  <xacro:property name="wheel_pos_y" value="0.14" />
   <xacro:property name="wheel_pos_z" value="-0.03" />
   <xacro:property name="wheel_mass" value=".1" />
   <xacro:property name="wheel_torque" value="20" />
-  <xacro:property name="front_caster_wheel" value="true" />
+  <xacro:property name="front_caster_wheel" value="false" />
   <xacro:property name="rear_caster_wheel" value="true" />
   <!-- set empty on the wheel_mesh_file to use geometry instead of mesh -->
@@ -21,5 +21,5 @@
   <!-- <xacro:property name="wheel_mesh_file" value="file://$(find linorobot2_description)/meshes/tire.dae" /> -->
   <xacro:property name="laser_pose">
-    <origin xyz="0.12 0 0.33" rpy="0 0 0"/>
+    <origin xyz="0 0 0.08" rpy="0 0 ${pi}"/>
   </xacro:property>
   <xacro:property name="depth_sensor_pose">

Commit message: Reversed the Lidar so front of the lidar is facing front of the robot

File: linorobot2_description/urdf/2wd_properties.urdf.xacro (robot description, xacro)
@@ -21,5 +21,8 @@
   <!-- <xacro:property name="wheel_mesh_file" value="file://$(find linorobot2_description)/meshes/tire.dae" /> -->
   <xacro:property name="laser_pose">
+<!-- Use this if your lidar's front is facing the rear:
     <origin xyz="0 0 0.08" rpy="0 0 ${pi}"/>
+-->
+    <origin xyz="0 0 0.08" rpy="0 0 0"/>
   </xacro:property>
   <xacro:property name="depth_sensor_pose">
